File: hardware/openuav.kicad_sch (KiCad schematic)
At the start: 66 parts, among them J1 Conn_01x01, J10 Conn_01x01, J11 Conn_01x01, J12 Conn_01x01, J13 Conn_01x01, J14 Conn_01x01, J19 Conn_01x01, J2 Conn_01x01, J20 Conn_01x01, J22 Conn_01x01, J23 Conn_01x01, J24 Conn_01x01, J25 Conn_01x01, J3 Conn_01x01, J30 Conn_01x01, J31 Conn_01x01, J4 Conn_01x01, J5 Conn_01x01, J6 Conn_01x01, J7 Conn_01x01, J8 Conn_01x01, J9 Conn_01x01, J99 USB_C_Receptacle_USB2.0, SW1 SW_Push, U1 STM32G431CBUx, U2 LPS22HH, U3 LSM6DSR, U4 TPS54302, U6 W25N01GVZEIG, U7 TLV75733PDBV

Commit message: Swap USB power diode for smaller part
Parts:
- D1: value SS34 -> PMEG2020AEA; footprint Diode_SMD:D_SMA -> Diode_SMD:D_SOD-323; LCSC C8678 -> C389354
Changed lines of the file:
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@@
   (symbol (lib_id "Device:D_Schottky_Small") (at 123.19 83.82 180) (unit 1)
     (in_bom yes) (on_board yes) (dnp no)
-    (property "Reference" "D1" (at 128.27 81.28 0)
+    (property "Reference" "D1" (at 123.19 79.375 0)
       (effects (font (size 1.27 1.27)))
     )
-    (property "Value" "SS34" (at 123.19 81.28 0)
+    (property "Value" "PMEG2020AEA" (at 123.19 81.28 0)
       (effects (font (size 1.27 1.27)))
     )
-    (property "Footprint" "Diode_SMD:D_SMA" (at 123.19 83.82 90)
+    (property "Footprint" "Diode_SMD:D_SOD-323" (at 123.19 83.82 90)
       (effects (font (size 1.27 1.27)) hide)
     )
@@
       (effects (font (size 1.27 1.27)) hide)
     )
-    (property "LCSC" "C8678" (at 123.19 83.82 0)
+    (property "LCSC" "C389354" (at 123.19 83.82 0)
       (effects (font (size 1.27 1.27)) hide)
     )

Commit message: Finish v3 board design
Parts:
- removed J30, J31: Conn_01x01, footprints:largepad, symbol Connector_Generic:Conn_01x01
- added C17, C18, C19, C20, C21, C22, C23, C8: 10u, Capacitor_SMD:C_0603_1608Metric, symbol Device:C
- added J15, J16, J17, J18, J21: Conn_01x01, footprints:smallpad, symbol Connector_Generic:Conn_01x01
- added R5: 10k, Resistor_SMD:R_0402_1005Metric, symbol Device:R_Small
- added U5: TLV75733PDBV, Package_TO_SOT_SMD:SOT-23-5, symbol Regulator_Linear:TLV75733PDBV
- C24, C25: value 1u -> 10u; footprint Capacitor_SMD:C_0402_1005Metric -> Capacitor_SMD:C_0603_1608Metric; LCSC C52923 -> C19702
Connections:
- net SWCLK is gone; now on net LED2: U1.37 (PA14)
- net SWDIO is gone; now on net LED1: U1.36 (PA13)
- net +3V3: now also C25.1, C23.1, C8.1, U5.3 (EN); no longer C3.1, U3.8 (Vdd)
- net +5V: now also C17.1, C18.1, C20.1, C21.1, C22.1, J18.1 (Pin_1), U5.1 (IN); no longer C25.1, J10.1 (Pin_1)
- net +BATT: now also J10.1 (Pin_1), J15.1 (Pin_1)
- net GND: now also U7.4 (NC), C17.2, C18.2, C19.2, C20.2, C21.2, C22.2, C23.2, C8.2, J16.1 (Pin_1), J17.1 (Pin_1), U5.2 (GND), U5.4 (NC)
- net LED1: no longer U1.47 (PB9)
- net LED2: no longer U1.32 (PA10)
- net SPI3_CS: now also U1.47 (PB9); no longer U1.38 (PA15)
- net VOLTAGE: no longer U1.5 (PF0)
- new net CSENSE: R5.2, U1.5 (PF0)
- new net CURRENT: J21.1 (Pin_1), R5.1
- new net VDDA: C19.1, C3.1, U3.8 (Vdd), U5.5 (OUT)
Other:
- note added: "Additional Capacitors"
- moved on the sheet: C11, C3, J13, J14, R8, SW1
