File: esc/esc.kicad_sch (KiCad schematic)
At the start: 34 parts, among them Q1 BSC0702LS, Q2 BSC0702LS, Q3 BSC0702LS, Q4 BSC0702LS, Q5 BSC0702LS, Q6 BSC0702LS, U1 AT32F421G8U7, U2 DRV8300, U3 INA180A

Commit message: Continued work on ESC
Parts:
- removed C1: 100n, symbol Device:C_Small
- removed C2, C3, C4: 1u, symbol Device:C_Small
- removed D1, D2, D3: D, symbol Device:D_Schottky_Small
- removed Q1, Q2, Q3, Q4, Q5, Q6: BSC0702LS, Package_TO_SOT_SMD:TDSON-8-1, symbol Transistor_FET:BSC070N10NS5
- removed R1, R10, R13, R16: 1k, symbol Device:R_Small
- removed R11, R12, R14, R15, R8, R9: 10k, symbol Device:R_Small
- removed R2, R3, R4, R5, R6, R7: 10, symbol Device:R_Small
- removed U1: AT32F421G8U7, Package_DFN_QFN:QFN-28_4x4mm_P0.5mm, symbol MCU_ST_STM32F0:STM32F031G4Ux
- removed U2: DRV8300, Package_DFN_QFN:HVQFN-24-1EP_4x4mm_P0.5mm_EP2.5x2.5mm_ThermalVias, symbol ESC:DRV8300
- added C10: 47u, Capacitor_SMD:C_1210_3225Metric, symbol Device:C
- added C11: 100n, symbol Device:C_Small
- added C5, C6: 10u, Capacitor_SMD:C_0603_1608Metric, symbol Device:C
- added C7: 100n, Capacitor_SMD:C_0402_1005Metric, symbol Device:C_Small
- added C8: 68p, Capacitor_SMD:C_0402_1005Metric, symbol Device:C_Small
- added C9: 10u, Capacitor_SMD:C_1206_3216Metric, symbol Device:C
- added D4: LED, symbol Device:LED
- added H1, H2, H3, H4: MountingHole, MountingHole:MountingHole_4mm, symbol Mechanical:MountingHole
- added L1: 10u, Inductor_SMD:L_Sunlord_MWSA0503S, symbol Device:L_Small
- added R17: 100k, Resistor_SMD:R_0402_1005Metric, symbol Device:R_Small
- added R18: 100k, symbol Device:R_Small
- added R19: 10k, symbol Device:R_Small
- added R22: R, Resistor_SMD:R_0402_1005Metric, symbol Device:R_Small
- added R23: 1k, symbol Device:R_Small
- added U3: TLV75733PDBV, Package_TO_SOT_SMD:SOT-23-5, symbol Regulator_Linear:TLV75733PDBV
- added U4: TPS54302, Package_TO_SOT_SMD:SOT-23-6, symbol Regulator_Switching:TPS54302
- renumbered R17 to R20, R18 to R21, U3 to U5
Connections:
- net +3V3: now also C6.1, R23.1, U3.5 (OUT)
- net +5V: now also C5.1, U3.1 (IN), U3.3 (EN)
- net +BATT: now also C9.1, R18.1, U4.3 (VIN)
- net CURRENT: now also C11.1
- net GND: now also C10.2, C11.2, C5.2, C6.2, C9.2, D4.1 (K), R19.2, R22.2, U3.2 (GND), U3.4 (NC), U4.1 (GND)
- net VSENSE: now also R18.2, R19.1
- net SOURCE: now reaches R20.1, U5.3 (+)
- new net: C8.1, R17.2, R22.1, U4.4 (FB)
- new net: C7.2, L1.1, U4.2 (SW)
- new net: C7.1, U4.6 (BOOT)
- new net: D4.2 (A), R23.2
- new net +9V: C10.1, C8.2, L1.2, R17.1
- no-connect marks 8 -> 1
Other:
- added sheet Single ESC 1 (single_esc.kicad_sch)
- added sheet Single ESC2 (single_esc.kicad_sch)
- added sheet Single ESC3 (single_esc.kicad_sch)
- added sheet Single ESC4 (single_esc.kicad_sch)
- moved on the sheet: R20, R21, U5
